File: coin-trunker/USBCon.sch (KiCad schematic (older format))
At the start: 11 parts, among them J6 Conn_01x05, J7 USB_B_Micro, U6 MCP1703A-3302_SOT23, U7 STM32F042F6Px

Commit message: Release version 0.1.0
Parts:
- J7: symbol Connector:USB_B_Micro -> coin-trunker-rescue:USB_B_Micro-Connector
- U7: symbol MCU_ST_STM32F0:STM32F042F6Px -> coin-trunker-rescue:STM32F042F6Px-MCU_ST_STM32F0
Changed lines of the file:
@@
 $EndDescr
 $Comp
-L MCU_ST_STM32F0:STM32F042F6Px U7
+L coin-trunker-rescue:STM32F042F6Px-MCU_ST_STM32F0 U7
 U 1 1 5FE0C064
 P 4650 2800
@@
 $EndComp
 $Comp
-L Connector:USB_B_Micro J7
+L coin-trunker-rescue:USB_B_Micro-Connector J7
 U 1 1 5FE0CA19
 P 7850 2800
